File: input.kicad_sch (KiCad schematic)
At the start: 46 parts, among them U10 PC817, U11 PC817, U12 PC817, U13 PC817, U14 PC817, U15 PC817, U16 PC817, U17 PC817, U18 ACS712xLCTR-05B, U5 PC817, U6 PC817, U7 PC817, U8 PC817, U9 PC817

Commit message: change references
Parts:
- renumbered C21 to C10, C9 to C11, C14 to C12, C19 to C13, C22 to C14, C10 to C15, C15 to C16, C20 to C17, C23 to C18, C11 to C19, C12 to C20, C16 to C21, C17 to C22, C1 to C7, C13 to C8, C18 to C9, R22 to R10, R10 to R11, R14 to R12, R20 to R13, R23 to R14, R11 to R15, R15 to R16, R16 to R18, R1 to R3, R12 to R4, R18 to R5, R21 to R6, R9 to R7, R13 to R8, R19 to R9

Commit message: add C values
Parts:
- C10, C11, C12, C13, C14, C15, C16, C17, C18, C19, C20, C7, C8, C9: value C -> 100nF
- C21: value C -> 1nF
