File: output.kicad_sch (KiCad schematic)
At the start: 60 parts, among them Q1 BC847, Q10 BC847, Q2 BC847, Q3 BC847, Q4 BC847, Q5 BC847, Q6 BC847, Q7 BC847, Q8 BC847, Q9 BC847, U19 PC817, U20 PC817, U21 PC817, U22 PC817, U23 PC817, U24 PC817, U25 PC817, U26 PC817, U27 PC817, U28 PC817

Commit message: change references
Parts:
- renumbered R2 to R19, R4 to R20, R3 to R21, R24 to R22, R25 to R23, R26 to R24, R27 to R25, R28 to R26, R29 to R27, R30 to R28, R31 to R29, R32 to R30, R33 to R31, R34 to R32, R35 to R33, R36 to R34, R37 to R35, R38 to R36, R39 to R37, R40 to R38, R41 to R39, R42 to R40, R43 to R41, R44 to R42, R45 to R43, R46 to R44, R47 to R45, R48 to R46, R49 to R47, R50 to R48

Commit message: update project to kicad 9
Parts:
- removed D1, D10, D11, D3, D4, D5, D6, D7, D8, D9: 1N4007, Diode_SMD:D_SMA_Handsoldering, symbol Diode:1N4007
- added D1, D10, D2, D3, D4, D5, D6, D7, D8, D9: 1N4148W, Diode_SMD:D_SOD-123, symbol Diode:1N4148W
Connections:
- net +24V: now also D1.1 (K), D10.1 (K), D2.1 (K), D3.1 (K), D4.1 (K), D5.1 (K), D6.1 (K), D7.1 (K), D8.1 (K), D9.1 (K)
- net DO1: now also D1.2 (A)
- net DO10: now also D10.2 (A)
- net DO2: now also D2.2 (A)
- net DO3: now also D3.2 (A)
- net DO4: now also D4.2 (A)
- net DO5: now also D5.2 (A)
- net DO6: now also D6.2 (A)
- net DO7: now also D7.2 (A)
- net DO8: now also D8.2 (A)
- net DO9: now also D9.2 (A)
