File: industrial-board.kicad_pcb (KiCad board)
At the start: 2 copper layers, 100 x 100 mm, 131 parts, among them J1 Conn_01x06_Pin, J2 Conn_01x14, J3 Conn_01x15, J4 Conn_01x04, J5 Conn_01x03, Q1 BC847, Q10 BC847, Q2 BC847, Q3 BC847, Q4 BC847, Q5 BC847, Q6 BC847, Q7 BC847, Q8 BC847, Q9 BC847, SW1 SW_Push, U1 STM32F103C8Tx, U10 PC817, U11 PC817, U12 PC817, U13 PC817, U14 PC817, U15 PC817, U16 PC817, U17 PC817, U18 ACS712xLCTR-05B, U19 PC817, U2 AMS1117-3.3, U20 PC817, U21 PC817, U22 PC817, U23 PC817, U24 PC817, U25 PC817, U26 PC817, U27 PC817, U28 PC817, U3 PEAK P6CU-2405ELF, U4 MAX3485, U5 PC817, U6 PC817, U7 PC817, U8 PC817, U9 PC817, Y1 8MHz, Y2 32KHz

Commit message: change references
Parts:
- renumbered BT2 to BT1, C5 to C1, C21 to C10, C9 to C11, C14 to C12, C19 to C13, C22 to C14, C10 to C15, C15 to C16, C20 to C17, C23 to C18, C11 to C19, C6 to C2, C12 to C20, C16 to C21, C17 to C22, C7 to C3, C8 to C4, C24 to C5, C3 to C6, C1 to C7, C13 to C8, C18 to C9, J3 to J2, J5 to J3, J2 to J4, J4 to J5, R51 to R1, R22 to R10, R10 to R11, R14 to R12, R20 to R13, R23 to R14, R11 to R15, R15 to R16, R16 to R18, R2 to R19, R7 to R2, R4 to R20, R3 to R21, R24 to R22, R25 to R23, R26 to R24, R27 to R25, R28 to R26, R29 to R27, R30 to R28, R31 to R29, R1 to R3, R32 to R30, R33 to R31, R34 to R32, R35 to R33, R36 to R34, R37 to R35, R38 to R36, R39 to R37, R40 to R38, R41 to R39, R12 to R4, R42 to R40, R43 to R41, R44 to R42, R45 to R43, R46 to R44, R47 to R45, R48 to R46, R49 to R47, R50 to R48, R18 to R5, R21 to R6, R9 to R7, R13 to R8, R19 to R9
Routing:
- net /IP-: track 8.83 -> 10.4 mm
- net /IP+: track 9.15 -> 10.2 mm

Commit message: minor changes
Parts:
- moved R1 28.4 mm to (75.0, 102.2), turned to 180 degrees
- moved C5 13.8 mm to (108.5, 87.5), turned to 90 degrees
- moved C4 1.51 mm to (90.0, 83.5)
- moved C3 1.51 mm to (99.0, 83.4)
- moved Y2 1.51 mm to (93.2, 84.4)
- moved Y1 1.50 mm to (94.6, 92.5)
- moved C1 1.46 mm to (99.2, 87.8)
- moved C2 1.46 mm to (89.8, 87.8)
Connections:
- J3 pad 1: /RS485+ -> /RS485-
- J3 pad 2: /RS485- -> /RS485+
Routing:
- net /NRST: track 80.2 -> 88.1 mm, vias 3 -> 4
- net /RS485+: track 35.7 -> 29.7 mm
- net /CLK_OSC_IN: track 21.6 -> 18.4 mm
- net /CLK_OSC_OUT: track 27.6 -> 24.5 mm
- net +3.3V: track 152.4 -> 154.9 mm, vias 5 -> 2
- net /RX: track 43.4 -> 41.1 mm, vias 2 -> 0
- net /TX: track 47.2 -> 45.0 mm, vias 2 -> 0
- net /OSC_OUT: track 26.5 -> 25.3 mm
- net /TX_EN: track 45.1 -> 46.2 mm, vias 2 -> 0
- net GND: track 18.2 -> 17.0 mm, vias 5 -> 6
- net /OSC_IN: track 14.2 -> 13.1 mm
- net /SWDCLK: track 34.9 -> 34.1 mm, vias 0 -> 2
- net /JTDO: vias 0 -> 2
- net /SWDIO: vias 0 -> 2

Commit message: add C values
Parts:
- C10, C11, C12, C13, C14, C15, C16, C17, C18, C19, C7, C8, C9: value C -> 100nF
- C5: value C -> 1uF
- C6: value C -> 10uF
Changed lines of the file:
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@@
 			)
 		)
-		(property "Value" "C"
+		(property "Value" "100nF"
 			(at 2.5 0 0)
 			(layer "F.Fab")
@@
 			)
 		)
-		(property "Value" "C"
+		(property "Value" "100nF"
 			(at 2.5 0 0)
 			(layer "F.Fab")
@@
 			)
 		)
-		(property "Value" "C"
+		(property "Value" "100nF"
 			(at 2.5375 0 0)
 			(layer "F.Fab")
@@
 			)
 		)
-		(property "Value" "C"
+		(property "Value" "100nF"
 			(at 2.5 0 0)
 			(layer "F.Fab")
@@
 			)
 		)
-		(property "Value" "C"
+		(property "Value" "100nF"
 			(at 2.5 0 0)
 			(layer "F.Fab")
@@
 			)
 		)
-		(property "Value" "C"
+		(property "Value" "100nF"
 			(at 2.5 0 0)
 			(layer "F.Fab")
@@
 			)
 		)
-		(property "Value" "C"
+		(property "Value" "100nF"
 			(at 2.4625 0 0)
 			(layer "F.Fab")
@@
 			)
 		)
-		(property "Value" "C"
+		(property "Value" "100nF"
 			(at 2.5 0 0)
 			(layer "F.Fab")
@@
 			)
 		)
-		(property "Value" "C"
+		(property "Value" "10uF"
 			(at 0 1.68 90)
 			(layer "F.Fab")
@@
 			)
 		)
-		(property "Value" "C"
+		(property "Value" "100nF"
 			(at 2.4625 0 0)
 			(layer "F.Fab")
@@
 			)
 		)
-		(property "Value" "C"
+		(property "Value" "100nF"
 			(at 2.5 0 0)
 			(layer "F.Fab")
@@
 			)
 		)
-		(property "Value" "C"
+		(property "Value" "100nF"
 			(at 2.5 0 0)
 			(layer "F.Fab")
@@
 			)
 		)
-		(property "Value" "C"
+		(property "Value" "100nF"
 			(at 2.5 0 0)
 			(layer "F.Fab")
@@
 			)
 		)
-		(property "Value" "C"
+		(property "Value" "100nF"
 			(at 2.5 0 0)
 			(layer "F.Fab")
@@
 			)
 		)
-		(property "Value" "C"
+		(property "Value" "1uF"
 			(at 0 -1.5 90)
 			(layer "F.Fab")

Commit message: move components
Parts:
- C20: value C -> 100nF
- C21: value C -> 1nF
- moved C9 3.76 mm to (65.8, 62.2), turned to 90 degrees
- moved C8 3.69 mm to (59.2, 62.2), turned to 90 degrees
- moved C11 3.66 mm to (78.8, 62.3), turned to 90 degrees
- moved C7 3.65 mm to (52.8, 62.3), turned to 90 degrees
- moved C10 3.59 mm to (72.2, 62.2), turned to 90 degrees
- moved C14 3.58 mm to (98.2, 62.2), turned to 90 degrees
- moved C17 3.57 mm to (117.7, 62.2), turned to 90 degrees
- moved C18 3.57 mm to (124.2, 62.2), turned to 90 degrees
- moved C19 3.57 mm to (130.7, 62.2), turned to 90 degrees
- moved C13 3.57 mm to (91.8, 62.2), turned to 90 degrees
- moved C15 3.57 mm to (104.8, 62.2), turned to 90 degrees
- moved C16 3.57 mm to (111.2, 62.2), turned to 90 degrees
- moved C12 3.55 mm to (85.2, 62.2), turned to 90 degrees
- moved U10 2.25 mm to (88.3, 67.0)
- moved U11 2.25 mm to (94.8, 67.0)
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Routing:
- net /DI8: track 10.9 -> 13.2 mm
- net /IN5: track 45.2 -> 47.5 mm
- net /IN9: track 15.1 -> 17.3 mm
- net /IN10: track 15.3 -> 17.5 mm
- net /DI12: track 23.2 -> 25.2 mm
- net /DI13: track 26.2 -> 28.2 mm
- net /DI9: track 14.2 -> 16.2 mm
- net /DI11: track 20.2 -> 22.2 mm
- net /DI10: track 17.2 -> 19.2 mm
- net /DI3: track 9.51 -> 11.2 mm
- net /IN1: track 74.9 -> 76.6 mm
- net Net-(C10-Pad1): track 8.73 -> 7.08 mm
- net /IN3: track 60.2 -> 61.8 mm
- net /IN2: track 67.6 -> 69.1 mm
- net /DI4: track 8.35 -> 6.81 mm
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
Commit message: minor changes
Routing:
- net /NRST: track 88.1 -> 87.5 mm
Changed lines of the file:
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@@
 			(plot_on_all_layers_selection 0x0000000_00000000)
 			(disableapertmacros no)
-			(usegerberextensions no)
-			(usegerberattributes yes)
-			(usegerberadvancedattributes yes)
-			(creategerberjobfile yes)
+			(usegerberextensions yes)
+			(usegerberattributes no)
+			(usegerberadvancedattributes no)
+			(creategerberjobfile no)
 			(dashed_line_dash_ratio 12.000000)
 			(dashed_line_gap_ratio 3.000000)
@@
 			(psa4output no)
 			(plotreference yes)
-			(plotvalue yes)
+			(plotvalue no)
 			(plotfptext yes)
 			(plotinvisibletext no)
 			(sketchpadsonfab no)
-			(subtractmaskfromsilk no)
+			(subtractmaskfromsilk yes)
 			(outputformat 1)
 			(mirror no)
-			(drillshape 1)
+			(drillshape 0)
 			(scaleselection 1)
-			(outputdirectory "")
+			(outputdirectory "gerber/")
 		)
 	)
@@
 	)
 	(segment
+		(start 109.15 95.252233)
+		(end 108.652233 95.75)
+		(width 0.2)
+		(layer "F.Cu")
+		(net 3)
+	)
+	(segment
 		(start 110.75 92.25)
 		(end 110.75 90.8375)
@@
 	)
 	(segment
-		(start 109.15 95.055938)
-		(end 108.455938 95.75)
-		(width 0.2)
-		(layer "F.Cu")
-		(net 3)
-	)
-	(segment
 		(start 109.25 90.8375)
 		(end 109.25 91.75)
@@
 	)
 	(segment
-		(start 74.5 133)
-		(end 74.5 129)
+		(start 108.652233 95.75)
+		(end 107.3375 95.75)
 		(width 0.2)
 		(layer "F.Cu")
@@
 	)
 	(segment
-		(start 113.75 101.25)
-		(end 113.75 99.1625)
+		(start 74.5 133)
+		(end 74.5 129)
 		(width 0.2)
 		(layer "F.Cu")
@@
 	)
 	(segment
-		(start 108.455938 95.75)
-		(end 107.3375 95.75)
+		(start 113.75 101.25)
+		(end 113.75 99.1625)
 		(width 0.2)
 		(layer "F.Cu")
@@
 	)
 	(via
-		(at 109.15 95.055938)
+		(at 109.15 95.252233)
 		(size 0.6)
 		(drill 0.3)
@@
 	)
 	(segment
+		(start 108.303705 95.25)
+		(end 107.3375 95.25)
+		(width 0.2)
+		(layer "F.Cu")
+		(net 68)
+	)
+	(segment
 		(start 107.3125 95.225)
 		(end 85.825 95.225)
@@
 	)
 	(segment
-		(start 108.75 93.75)
-		(end 108.75 94.60741)
-		(width 0.2)
-		(layer "F.Cu")
-		(net 68)
-	)
-	(segment
-		(start 108.75 94.60741)
-		(end 108.10741 95.25)
-		(width 0.2)
-		(layer "F.Cu")
-		(net 68)
-	)
-	(segment
 		(start 144.75 100.5)
 		(end 146.5 100.5)
@@
 	)
 	(segment
+		(start 109.053705 94.303705)
+		(end 109.053705 94.5)
+		(width 0.2)
+		(layer "F.Cu")
+		(net 68)
+	)
+	(segment
 		(start 138.300003 94.050003)
 		(end 144.75 100.5)
@@
 	)
 	(segment
-		(start 108.10741 95.25)
-		(end 107.3375 95.25)
+		(start 74 102.25)
+		(end 74 94)
 		(width 0.2)
 		(layer "F.Cu")
@@
 	)
 	(segment
-		(start 74 102.25)
-		(end 74 94)
+		(start 109.053705 94.5)
+		(end 108.303705 95.25)
 		(width 0.2)
 		(layer "F.Cu")
@@
 	)
 	(via
-		(at 108.75 93.75)
+		(at 109.053705 94.303705)
 		(size 0.6)
 		(drill 0.3)
@@
 	)
 	(segment
-		(start 108.75 93.75)
-		(end 116.901471 93.75)
+		(start 109.307407 94.050003)
+		(end 119.5 94.050003)
 		(width 0.2)
 		(layer "B.Cu")
@@
 	)
 	(segment
-		(start 116.901471 93.75)
-		(end 117.201474 94.050003)
-		(width 0.2)
-		(layer "B.Cu")
-		(net 68)
-	)
-	(segment
-		(start 117.201474 94.050003)
-		(end 119.5 94.050003)
+		(start 109.053705 94.303705)
+		(end 109.307407 94.050003)
 		(width 0.2)
 		(layer "B.Cu")
@@
 		(polygon
 			(pts
-				(xy 50 69.5) (xy 51 69.5) (xy 51 133.5) (xy 50 133.5)
+				(xy 50 69.25) (xy 51.25 69.25) (xy 51.25 133.5) (xy 50 133.5)
 			)
 		)

Commit message: update project to kicad 9
Parts:
- removed D11: 1N4007, Diode_SMD:D_SMA_Handsoldering
- added D2: 1N4148W, Diode_SMD:D_SOD-123, F.Cu at (91.5, 136.8)
- D1, D10, D3, D4, D5, D6, D7, D8, D9: value 1N4007 -> 1N4148W; footprint Diode_SMD:D_SMA_Handsoldering -> Diode_SMD:D_SOD-123
- H1, H2, H3, H4: footprint MountingHole:MountingHole_4.3mm_M4 -> MountingHole:MountingHole_3.2mm_M3
- moved H1 92.0 mm to (53.5, 146.5)
- moved H2 92.0 mm to (53.5, 53.5)
- moved H3 92.0 mm to (146.5, 53.5)
- moved H4 92.0 mm to (146.5, 146.5)
- moved D5 5.10 mm to (106.5, 137.0)
- moved D10 5.07 mm to (131.5, 136.8)
- moved D3 5.07 mm to (96.5, 136.8)
- moved D6 5.07 mm to (111.5, 136.8)
- moved D7 5.07 mm to (116.5, 136.8)
- moved D8 5.07 mm to (121.5, 136.8)
- moved D9 5.07 mm to (126.5, 136.8)
- moved D4 4.96 mm to (101.4, 136.8)
- moved D1 0.85 mm to (86.5, 136.8)
Connections:
- D10 pad 2: /DO9 -> /DO10
- D3 pad 2: /DO2 -> /DO3
- D4 pad 2: /DO3 -> /DO4
- D5 pad 2: /DO4 -> /DO5
- D6 pad 2: /DO5 -> /DO6
- D7 pad 2: /DO6 -> /DO7
- D8 pad 2: /DO7 -> /DO8
- D9 pad 2: /DO8 -> /DO9
Routing:
- net +24V: track 198.7 -> 212.6 mm

Commit message: ground crystal oscillators
Connections:
- C1 pad 1: Net-(C1-Pad1) -> GND
- C2 pad 1: Net-(C1-Pad1) -> GND
- C3 pad 1: Net-(C3-Pad1) -> GND
- C4 pad 1: Net-(C3-Pad1) -> GND
Routing:
- net Net-(C3-Pad1): track 9.02 -> 0.00 mm
- net Net-(C1-Pad1): track 7.43 -> 0.00 mm
